Commit message: update urdf can change load

File: assets/nezha/urdf/nezha.urdf (robot description, URDF)
Before this commit: robot nezha, 22 links, 21 joints
Links:
- added link imu_fixed_link, mass 0.0406912140939172; visual mesh filename=../meshes/imu_fixed_joint.STL
- added link top_box, mass 0.0; collision box size=0.5 0.35 0.08; visual box size=0.5 0.35 0.15
- link FL_calf: mass 0.65961881 -> 0.8; geometry collision box size=0.05 0.045 0.390; visual mesh filename=../meshes/FL_calf.STL
- link FL_foot: geometry collision cylinder length=0.040 radius=0.105; visual mesh filename=../meshes/FL_foot.STL
- link FL_footmotor: mass 1.0 -> 1
- link FL_hip: mass 2.37707148 -> 3.1; geometry visual mesh filename=../meshes/FL_hip.STL
- link FL_thigh: mass 4.32911658 -> 4.1; geometry visual mesh filename=../meshes/FL_thigh.STL
- link FR_calf: mass 0.65961882 -> 0.8; geometry collision box size=0.05 0.045 0.390; visual mesh filename=../meshes/FR_calf.STL
- link FR_foot: geometry collision cylinder length=0.040 radius=0.105; visual mesh filename=../meshes/FR_foot.STL
- link FR_footmotor: mass 1.0 -> 1
- link FR_hip: mass 2.37707148 -> 3.1; geometry visual mesh filename=../meshes/FR_hip.STL
- link FR_thigh: mass 4.32961796 -> 4.1; geometry visual mesh filename=../meshes/FR_thigh.STL
- link Lidar: mass 0.81416515 -> 1; geometry visual mesh filename=../meshes/Lidar.STL
- link RL_calf: mass 0.65961881 -> 0.8; geometry collision box size=0.05 0.045 0.390; visual mesh filename=../meshes/RL_calf.STL
- link RL_foot: geometry collision cylinder length=0.040 radius=0.105; visual mesh filename=../meshes/RL_foot.STL
- link RL_footmotor: mass 1.0 -> 1
- link RL_hip: mass 2.37707148 -> 3.1; geometry visual mesh filename=../meshes/RL_hip.STL
- link RL_thigh: mass 4.32911658 -> 4.1; geometry visual mesh filename=../meshes/RL_thigh.STL
- link RR_calf: mass 0.65961882 -> 0.8; geometry collision box size=0.05 0.045 0.390; visual mesh filename=../meshes/RR_calf.STL
- link RR_foot: geometry collision cylinder length=0.040 radius=0.105; visual mesh filename=../meshes/RR_foot.STL
- link RR_footmotor: mass 1.0 -> 1
- link RR_hip: mass 2.37707148 -> 3.1; geometry visual mesh filename=../meshes/RR_hip.STL
- link RR_thigh: mass 4.32961796 -> 4.1; geometry visual mesh filename=../meshes/RR_thigh.STL
- link trunk: mass 44.027 -> 37.6; geometry collision box size=1.121 0.390 0.27; visual mesh filename=../meshes/trunk.STL
Joints:
- added joint box_to_trunk_joint: type fixed, parent trunk, child top_box, origin xyz=0 -0.03 0.17 rpy=0 0 0
- added joint imu_fixed_joint: type fixed, parent trunk, child imu_fixed_link, origin xyz=0.00112019201975541 -0.0364882468746482 0.0510999999999999 rpy=0 0 0, axis 0 0 0
- joint FL_calf_joint: limit lower=-2.5 upper=-0.7 effort=225 velocity=8 -> lower=-2.3 upper=-0.52 effort=225 velocity=8; origin xyz=0 0.0245 -0.33 rpy=0 0 0 -> xyz=0 0.0241 -0.33 rpy=0 0 0
- joint FL_foot_joint: origin xyz=0.00010365 0.034479 0.00033954 rpy=0 0 0 -> xyz=0 0.067334 0.0052008 rpy=0 0 0
- joint FL_footmotor_fixed: origin xyz=5.7407E-05 0.0205 -0.33 rpy=0 0 0 -> xyz=0 -0.019084 -0.3352 rpy=0 0 0
- joint FL_hip_joint: limit lower=-0.6 upper=0.6 effort=150 velocity=12 -> lower=-1.31 upper=0.81 effort=150 velocity=12; origin xyz=0.42614 0.064917 0.013531 rpy=0 0 0 -> xyz=0.43304 0.056588 0.00014972 rpy=0 0 0
- joint FL_thigh_joint: limit lower=-0.3 upper=2.6 effort=150 velocity=12 -> lower=-1.5 upper=2.6 effort=150 velocity=12; origin xyz=0 0.1325 0 rpy=0 0 0 -> xyz=0 0.1324 0 rpy=0 0 0
- joint FR_calf_joint: limit lower=-2.5 upper=-0.7 effort=225 velocity=8 -> lower=-2.4 upper=-0.57 effort=225 velocity=8; origin xyz=0 -0.0245 -0.33 rpy=0 0 0 -> xyz=0 -0.0241 -0.33 rpy=0 0 0
- joint FR_foot_joint: origin xyz=7.9882E-05 -0.034479 0.0003459 rpy=0 0 0 -> xyz=0 -0.067334 0.0052008 rpy=0 0 0
- joint FR_footmotor_fixed: origin xyz=5.7407E-05 -0.0205 -0.33 rpy=0 0 0 -> xyz=0 0.019084 -0.3352 rpy=0 0 0
- joint FR_hip_joint: limit lower=-0.6 upper=0.6 effort=150 velocity=12 -> lower=-0.8 upper=1.3 effort=150 velocity=12; origin xyz=0.42614 -0.089083 0.013531 rpy=0 0 0 -> xyz=0.43304 -0.11341 0.00014972 rpy=0 0 0
- joint FR_thigh_joint: limit lower=-0.3 upper=2.6 effort=150 velocity=12 -> lower=-1.6 upper=2.6 effort=150 velocity=12; origin xyz=0 -0.1325 0 rpy=0 0 0 -> xyz=0 -0.1324 0 rpy=0 0 0
- joint Lidar_fixed_joint: axis 0 0 0 -> 1 0 0; origin xyz=0.56234 -0.012083 -0.027985 rpy=0 0 0 -> xyz=0.6019 -0.041631 0.032239 rpy=0 0 0
- joint RL_calf_joint: limit lower=-2.5 upper=-0.7 effort=225 velocity=8 -> lower=-2.6 upper=0.57 effort=225 velocity=8; origin xyz=0 0.0245 -0.33 rpy=0 0 0 -> xyz=0 0.0241 -0.33 rpy=0 0 0
- joint RL_foot_joint: origin xyz=0.00010365 0.034479 0.00033954 rpy=0 0 0 -> xyz=0 0.067334 0.0052008 rpy=0 0 0
- joint RL_footmotor_fixed: origin xyz=5.7407E-05 0.0205 -0.33 rpy=0 0 0 -> xyz=0 -0.019084 -0.3352 rpy=0 0 0
- joint RL_hip_joint: limit lower=-0.6 upper=0.6 effort=150 velocity=12 -> lower=-1.51 upper=0.8 effort=150 velocity=12; origin xyz=-0.43586 0.064917 0.013531 rpy=0 0 0 -> xyz=-0.42896 0.056588 0.00014972 rpy=0 0 0
- joint RL_thigh_joint: limit lower=-0.3 upper=2.6 effort=150 velocity=12 -> lower=-1.6 upper=2.6 effort=150 velocity=12; origin xyz=0 0.1325 0 rpy=0 0 0 -> xyz=0 0.1324 0 rpy=0 0 0
- joint RR_calf_joint: limit lower=-2.5 upper=-0.7 effort=225 velocity=8 -> lower=-2.6 upper=0.57 effort=225 velocity=8; origin xyz=0 -0.0245 -0.33 rpy=0 0 0 -> xyz=0 -0.0241 -0.33 rpy=0 0 0
- joint RR_foot_joint: origin xyz=7.9882E-05 -0.034479 0.0003459 rpy=0 0 0 -> xyz=0 -0.067334 0.0052008 rpy=0 0 0
- joint RR_footmotor_fixed: origin xyz=5.7407E-05 -0.0205 -0.33 rpy=0 0 0 -> xyz=0 0.019084 -0.3352 rpy=0 0 0
- joint RR_hip_joint: limit lower=-0.6 upper=0.6 effort=150 velocity=12 -> lower=-1.58 upper=0.79 effort=150 velocity=12; origin xyz=-0.43586 -0.089083 0.013531 rpy=0 0 0 -> xyz=-0.42896 -0.11341 0.00014972 rpy=0 0 0
- joint RR_thigh_joint: limit lower=-0.3 upper=2.6 effort=150 velocity=12 -> lower=-1.6 upper=2.6 effort=150 velocity=12; origin xyz=0 -0.1325 0 rpy=0 0 0 -> xyz=0 -0.1324 0 rpy=0 0 0

Commit message: Revert "update urdf can change load"
This reverts commit 43222cd70c567cf6499e2df2980a41c70b73f5e8.

File: assets/nezha/urdf/nezha.urdf (robot description, URDF)
Before this commit: robot nezha, 24 links, 23 joints
Links:
- removed link imu_fixed_link
- removed link top_box
- link FL_calf: mass 0.8 -> 0.65961881; geometry collision mesh filename=../meshes/FL_calf_collision.STL; visual mesh filename=../meshes/FL_calf.STL
- link FL_foot: geometry collision cylinder length=0.040 radius=0.11; visual mesh filename=../meshes/FL_foot.STL
- link FL_footmotor: mass 1 -> 1.0
- link FL_hip: mass 3.1 -> 2.37707148; geometry collision cylinder length=0.128 radius=0.065; visual mesh filename=../meshes/FL_hip.STL
- link FL_thigh: mass 4.1 -> 4.32911658; geometry collision mesh filename=../meshes/FL_thigh_collision.STL; visual mesh filename=../meshes/FL_thigh.STL
- link FR_calf: mass 0.8 -> 0.65961882; geometry collision mesh filename=../meshes/FR_calf_collision.STL; visual mesh filename=../meshes/FR_calf.STL
- link FR_foot: geometry collision cylinder length=0.040 radius=0.11; visual mesh filename=../meshes/FR_foot.STL
- link FR_footmotor: mass 1 -> 1.0
- link FR_hip: mass 3.1 -> 2.37707148; geometry collision cylinder length=0.128 radius=0.065; visual mesh filename=../meshes/FR_hip.STL
- link FR_thigh: mass 4.1 -> 4.32961796; geometry collision mesh filename=../meshes/FR_thigh_collision.STL; visual mesh filename=../meshes/FR_thigh.STL
- link Lidar: mass 1 -> 0.81416515; geometry collision box size=0.10 0.10 0.20; visual mesh filename=../meshes/Lidar.STL
- link RL_calf: mass 0.8 -> 0.65961881; geometry collision mesh filename=../meshes/FL_calf_collision.STL; visual mesh filename=../meshes/RL_calf.STL
- link RL_foot: geometry collision cylinder length=0.040 radius=0.11; visual mesh filename=../meshes/RL_foot.STL
- link RL_footmotor: mass 1 -> 1.0
- link RL_hip: mass 3.1 -> 2.37707148; geometry collision cylinder length=0.128 radius=0.065; visual mesh filename=../meshes/RL_hip.STL
- link RL_thigh: mass 4.1 -> 4.32911658; geometry collision mesh filename=../meshes/FL_thigh_collision.STL; visual mesh filename=../meshes/RL_thigh.STL
- link RR_calf: mass 0.8 -> 0.65961882; geometry collision mesh filename=../meshes/FR_calf_collision.STL; visual mesh filename=../meshes/RR_calf.STL
- link RR_foot: geometry collision cylinder length=0.040 radius=0.11; visual mesh filename=../meshes/RR_foot.STL
- link RR_footmotor: mass 1 -> 1.0
- link RR_hip: mass 3.1 -> 2.37707148; geometry collision cylinder length=0.128 radius=0.065; visual mesh filename=../meshes/RR_hip.STL
- link RR_thigh: mass 4.1 -> 4.32961796; geometry collision mesh filename=../meshes/FR_thigh_collision.STL; visual mesh filename=../meshes/RR_thigh.STL
- link trunk: mass 37.6 -> 44.027; geometry collision box size=0.70 0.34 0.20; visual mesh filename=../meshes/trunk.STL
Joints:
- removed joint box_to_trunk_joint
- removed joint imu_fixed_joint
- joint FL_calf_joint: limit lower=-2.3 upper=-0.52 effort=225 velocity=8 -> lower=-2.5 upper=-0.7 effort=225 velocity=8; origin xyz=0 0.0241 -0.33 rpy=0 0 0 -> xyz=0 0.0245 -0.33 rpy=0 0 0
- joint FL_foot_joint: origin xyz=0 0.067334 0.0052008 rpy=0 0 0 -> xyz=0.00010365 0.034479 0.00033954 rpy=0 0 0
- joint FL_footmotor_fixed: origin xyz=0 -0.019084 -0.3352 rpy=0 0 0 -> xyz=5.7407E-05 0.0205 -0.33 rpy=0 0 0
- joint FL_hip_joint: limit lower=-1.31 upper=0.81 effort=150 velocity=12 -> lower=-0.6 upper=0.6 effort=150 velocity=12; origin xyz=0.43304 0.056588 0.00014972 rpy=0 0 0 -> xyz=0.42614 0.064917 0.013531 rpy=0 0 0
- joint FL_thigh_joint: limit lower=-1.5 upper=2.6 effort=150 velocity=12 -> lower=-0.3 upper=2.6 effort=150 velocity=12; origin xyz=0 0.1324 0 rpy=0 0 0 -> xyz=0 0.1325 0 rpy=0 0 0
- joint FR_calf_joint: limit lower=-2.4 upper=-0.57 effort=225 velocity=8 -> lower=-2.5 upper=-0.7 effort=225 velocity=8; origin xyz=0 -0.0241 -0.33 rpy=0 0 0 -> xyz=0 -0.0245 -0.33 rpy=0 0 0
- joint FR_foot_joint: origin xyz=0 -0.067334 0.0052008 rpy=0 0 0 -> xyz=7.9882E-05 -0.034479 0.0003459 rpy=0 0 0
- joint FR_footmotor_fixed: origin xyz=0 0.019084 -0.3352 rpy=0 0 0 -> xyz=5.7407E-05 -0.0205 -0.33 rpy=0 0 0
- joint FR_hip_joint: limit lower=-0.8 upper=1.3 effort=150 velocity=12 -> lower=-0.6 upper=0.6 effort=150 velocity=12; origin xyz=0.43304 -0.11341 0.00014972 rpy=0 0 0 -> xyz=0.42614 -0.089083 0.013531 rpy=0 0 0
- joint FR_thigh_joint: limit lower=-1.6 upper=2.6 effort=150 velocity=12 -> lower=-0.3 upper=2.6 effort=150 velocity=12; origin xyz=0 -0.1324 0 rpy=0 0 0 -> xyz=0 -0.1325 0 rpy=0 0 0
- joint Lidar_fixed_joint: axis 1 0 0 -> 0 0 0; origin xyz=0.6019 -0.041631 0.032239 rpy=0 0 0 -> xyz=0.56234 -0.012083 -0.027985 rpy=0 0 0
- joint RL_calf_joint: limit lower=-2.6 upper=0.57 effort=225 velocity=8 -> lower=-2.5 upper=-0.7 effort=225 velocity=8; origin xyz=0 0.0241 -0.33 rpy=0 0 0 -> xyz=0 0.0245 -0.33 rpy=0 0 0
- joint RL_foot_joint: origin xyz=0 0.067334 0.0052008 rpy=0 0 0 -> xyz=0.00010365 0.034479 0.00033954 rpy=0 0 0
- joint RL_footmotor_fixed: origin xyz=0 -0.019084 -0.3352 rpy=0 0 0 -> xyz=5.7407E-05 0.0205 -0.33 rpy=0 0 0
- joint RL_hip_joint: limit lower=-1.51 upper=0.8 effort=150 velocity=12 -> lower=-0.6 upper=0.6 effort=150 velocity=12; origin xyz=-0.42896 0.056588 0.00014972 rpy=0 0 0 -> xyz=-0.43586 0.064917 0.013531 rpy=0 0 0
- joint RL_thigh_joint: limit lower=-1.6 upper=2.6 effort=150 velocity=12 -> lower=-0.3 upper=2.6 effort=150 velocity=12; origin xyz=0 0.1324 0 rpy=0 0 0 -> xyz=0 0.1325 0 rpy=0 0 0
- joint RR_calf_joint: limit lower=-2.6 upper=0.57 effort=225 velocity=8 -> lower=-2.5 upper=-0.7 effort=225 velocity=8; origin xyz=0 -0.0241 -0.33 rpy=0 0 0 -> xyz=0 -0.0245 -0.33 rpy=0 0 0
- joint RR_foot_joint: origin xyz=0 -0.067334 0.0052008 rpy=0 0 0 -> xyz=7.9882E-05 -0.034479 0.0003459 rpy=0 0 0
- joint RR_footmotor_fixed: origin xyz=0 0.019084 -0.3352 rpy=0 0 0 -> xyz=5.7407E-05 -0.0205 -0.33 rpy=0 0 0
- joint RR_hip_joint: limit lower=-1.58 upper=0.79 effort=150 velocity=12 -> lower=-0.6 upper=0.6 effort=150 velocity=12; origin xyz=-0.42896 -0.11341 0.00014972 rpy=0 0 0 -> xyz=-0.43586 -0.089083 0.013531 rpy=0 0 0
- joint RR_thigh_joint: limit lower=-1.6 upper=2.6 effort=150 velocity=12 -> lower=-0.3 upper=2.6 effort=150 velocity=12; origin xyz=0 -0.1324 0 rpy=0 0 0 -> xyz=0 -0.1325 0 rpy=0 0 0
